File: hardware/rotary/es_rotary.sch (KiCad schematic (older format))
At the start: 6 parts, among them J1 T3_Left, J2 T3_Right

Commit message: updated rot and display to v1.1
Parts:
- ROT1: footprint sparkfun:SF-ROTARY-ENCODER -> cvparts:Rotary_Encoder_PEC12R-3220F-S0024
Changed lines of the file:
@@
 F 0 "ROT1" H 2600 5037 60  0000 C CNN
 F 1 "ROTARY-ENCODER" H 2600 4931 60  0000 C CNN
-F 2 "sparkfun:SF-ROTARY-ENCODER" H 2600 4300 60  0000 C CNN
+F 2 "cvparts:Rotary_Encoder_PEC12R-3220F-S0024" H 2600 4100 60  0000 C CNN
 F 3 "" H 2600 4650 60  0000 C CNN
 	1    2600 4650
@@
 Connection ~ 3500 4750
 Text Label 4150 4550 0    50   ~ 0
+ENC_B
+Text Label 4150 4750 0    50   ~ 0
 ENC_A
-Text Label 4150 4750 0    50   ~ 0
-ENC_B
 Wire Wire Line
 	2050 3950 2050 3800
