File: hardware/display/es_display.kicad_pcb (KiCad board)
At the start: 2 copper layers, 40 x 72.4 mm, 8 parts, among them J1 T3_Left, J2 T3_Right, J3 OLED, J4 TFT

Commit message: updated rot and display to v1.1
Parts:
- moved J1 36.4 mm to (149.9, 104.1), turned to 180 degrees
- moved J2 36.4 mm to (134.6, 104.1), turned to 180 degrees
- renumbered REF** to Pad1, REF** to Pad2, REF** to Pad3, REF** to Pad4
Routing:
- net /CS: track 41.4 -> 96.6 mm, vias 0 -> 1
- net /MISO: track 46.4 -> 94.6 mm
- net /DSP_RST: track 36.5 -> 75.2 mm, vias 0 -> 2
- net /MOSI: track 61.4 -> 96.1 mm, vias 0 -> 1
- net /SCK: track 49.3 -> 83.8 mm
- net /DSP_C_S: track 43.6 -> 69.3 mm, vias 0 -> 1
- net /3.3V: track 105.7 -> 84.9 mm
- net GND: track 0.00 -> 10.7 mm, vias 1 -> 0
Other:
- board text added: "2o2o lallafa Rev 1.1"
- board text removed: "2o2o lallafa Rev 1.0"

Commit message: set license: CC-BY-SA-4.0
Other:
- board text added: "CC-BY-SA 4.0"
Changed lines of the file:
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@@
   (general
     (thickness 1.6)
-    (drawings 34)
+    (drawings 35)
     (tracks 69)
     (zones 0)
@@
   (page A4)
   (layers
-    (0 F.Cu signal)
-    (31 B.Cu signal)
+    (0 F.Cu signal hide)
+    (31 B.Cu signal hide)
     (32 B.Adhes user hide)
     (33 F.Adhes user hide)
@@
   )
   (setup
-    (last_trace_width 0.381)
+    (last_trace_width 0.25)
     (user_trace_width 0.254)
     (user_trace_width 0.381)
@@
     )
   )
+  (gr_text "CC-BY-SA\n4.0" (at 142.24 97.155) (layer F.SilkS)
+    (effects (font (size 1 1) (thickness 0.2) italic))
+  )
   (gr_text LITE (at 118.11 135.255) (layer F.SilkS)
     (effects (font (size 0.8 0.8) (thickness 0.15)))
@@
   (gr_line (start 112.395 140.97) (end 112.395 106.68) (layer Edge.Cuts) (width 0.05))
   (gr_line (start 152.4 140.97) (end 112.395 140.97) (layer Edge.Cuts) (width 0.05))
-  (gr_text "EuroShield\nDisplay Buddy" (at 142.24 87.63 270) (layer F.SilkS)
+  (gr_text "EuroShield\nDisplay Buddy" (at 142.24 85.09 270) (layer F.SilkS)
     (effects (font (size 1.5 1.5) (thickness 0.3)))
   )
-  (gr_text "2o2o\nlallafa\nRev 1.1" (at 142.24 73.66) (layer F.SilkS)
+  (gr_text "2o2o\nlallafa\nRev 1.1\n" (at 142.24 73.66) (layer F.SilkS)
     (effects (font (size 0.762 1.5) (thickness 0.1905)))
   )
