File: hardware/teensy4adapter/es_t4.kicad_pcb (KiCad board)
At the start: 2 copper layers, 22.9 x 38.1 mm, 5 parts, among them J1 T3_Left, J2 T3_Right, J3 T4_Left, J4 T4_Right

Commit message: set license: CC-BY-SA-4.0
Other:
- board text added: "CC-BY-SA 4.0"
Changed lines of the file:
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@@
   (general
     (thickness 1.6)
-    (drawings 27)
+    (drawings 28)
     (tracks 74)
     (zones 0)
@@
   (page A4)
   (layers
-    (0 F.Cu signal)
+    (0 F.Cu signal hide)
     (31 B.Cu signal)
     (32 B.Adhes user)
@@
     )
   )
+  (gr_text "CC-BY-SA\n4.0" (at 140.97 91.44) (layer F.SilkS)
+    (effects (font (size 1 1) (thickness 0.2)))
+  )
   (gr_text "2o2o\nlallafa\nRev 1.1" (at 140.97 101.6) (layer F.SilkS)
     (effects (font (size 0.762 1.5) (thickness 0.1905)))
   )
-  (gr_text "EuroShield\nTeensy 4\nAdapter" (at 140.97 85.09 90) (layer F.SilkS)
+  (gr_text "EuroShield\nTeensy 4\nAdapter" (at 140.97 82.55 90) (layer F.SilkS)
     (effects (font (size 1.5 1.5) (thickness 0.3)))
   )
